Commit message: 5.8雷达在中心可转到目标方向

File: src/tri_steer_description/urdf/tri_steer.xacro (robot description, xacro)
@@ -557,5 +557,5 @@
     <child link="laser"/>
     <!-- 例：雷达在车体前方 0.20m，高 0.12m -->
-    <origin xyz="0.0 0 0.3" rpy="0 0 0"/>
+    <origin xyz="0.0 0 0.12" rpy="0 0 0"/>
     <!-- <origin xyz="0.0 0.5 0.0" rpy="0 0 0"/> -->
     <!-- <origin xyz="0.0 0.5 0.0" rpy="1.5708 0 0"/> -->

Commit message: 5.11 雷达在车前并保持平稳转动,且不偏离终点

File: src/tri_steer_description/urdf/tri_steer.xacro (robot description, xacro)
@@ -557,5 +557,5 @@
     <child link="laser"/>
     <!-- 例：雷达在车体前方 0.20m，高 0.12m -->
-    <origin xyz="0.0 0 0.12" rpy="0 0 0"/>
+    <origin xyz="0.25 0 0.12" rpy="0 0 0"/>
     <!-- <origin xyz="0.0 0.5 0.0" rpy="0 0 0"/> -->
     <!-- <origin xyz="0.0 0.5 0.0" rpy="1.5708 0 0"/> -->
